File: ef936x_adapter.kicad_sch (KiCad schematic)
At the start: 5 parts, among them J1 Conn_01x20_Male, J2 Conn_01x20_Male, U1 EF9367, U2 74HC00, U3 74HC02

Commit message: Footprint fix
-footprint of EF9367 set to be a socket
-renamed schematic pdf file to be in line with other repos
Parts:
- U1: footprint Package_DIP:DIP-40_W15.24mm -> ef936x_adapter_lib_fp:DIP-40_W15.24mm_Socket
Changed lines of the file:
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@@
       (effects (font (size 1.27 1.27)) (justify left))
     )
-    (property "Footprint" "Package_DIP:DIP-40_W15.24mm" (at 67.31 48.26 0)
+    (property "Footprint" "ef936x_adapter_lib_fp:DIP-40_W15.24mm_Socket" (at 67.31 48.26 0)
       (effects (font (size 1.27 1.27)) hide)
     )
